File: BonkSwitch_hardware/BonkSwitch.sch (EAGLE design)
At the start: 96 parts, among them IC1 LMR16030SDDAR, IC2 LMR16006XDDC, IC3 FAN3227TMX, IC4 LMP8640MK-T, IC5 LMP8640MK-T, IC6 74LVC1G14DBV, Q1 SI2302CDS, T1 IRF7493TRPBF, T2 IRF7493TRPBF, X1 XT60PW-M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

Commit message: Adding Zener part numbers
Parts:
- D1, D4: MF (none) -> ON SEMICONDUCTOR; MPN (none) -> MM3Z4V3ST1G; OC_FARNELL unknown -> 2844819; OC_RS (none) -> 802-4625
Changed lines of the file:
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@@
 <part name="GND3" library="supply1" deviceset="GND" device=""/>
 <part name="D1" library="SparkFun-DiscreteSemi" deviceset="DIODE-ZENER" device="-MMSZ5232BS" value="5.6V">
-<attribute name="MF" value=""/>
-<attribute name="MPN" value=""/>
-<attribute name="OC_FARNELL" value="unknown"/>
+<attribute name="MF" value="ON SEMICONDUCTOR"/>
+<attribute name="MPN" value="MM3Z4V3ST1G"/>
+<attribute name="OC_FARNELL" value="2844819"/>
+<attribute name="OC_RS" value="802-4625"/>
 </part>
 <part name="GND6" library="supply1" deviceset="GND" device=""/>
@@
 <part name="GND11" library="supply1" deviceset="GND" device=""/>
 <part name="D4" library="SparkFun-DiscreteSemi" deviceset="DIODE-ZENER" device="-MMSZ5232BS" value="5.6V">
-<attribute name="MF" value=""/>
-<attribute name="MPN" value=""/>
-<attribute name="OC_FARNELL" value="unknown"/>
+<attribute name="MF" value="ON SEMICONDUCTOR"/>
+<attribute name="MPN" value="MM3Z4V3ST1G"/>
+<attribute name="OC_FARNELL" value="2844819"/>
+<attribute name="OC_RS" value="802-4625"/>
 </part>
 <part name="GND12" library="supply1" deviceset="GND" device=""/>
@@
 <attribute name="MF" x="33.02" y="116.84" size="1.778" layer="96" display="off"/>
 <attribute name="MPN" x="33.02" y="116.84" size="1.778" layer="96" display="off"/>
+<attribute name="OC_RS" x="33.02" y="116.84" size="1.778" layer="96" rot="R90" display="off"/>
 </instance>
 <instance part="GND6" gate="1" x="33.02" y="106.68"/>
@@
 <attribute name="MF" x="88.9" y="116.84" size="1.778" layer="96" display="off"/>
 <attribute name="MPN" x="88.9" y="116.84" size="1.778" layer="96" display="off"/>
+<attribute name="OC_RS" x="88.9" y="116.84" size="1.778" layer="96" rot="R90" display="off"/>
 </instance>
 <instance part="GND12" gate="1" x="88.9" y="106.68"/>
